File: PCB/LoRa_RFM98W_Shield.sch (EAGLE design)
At the start: 38 parts, among them IC1 SHT20, IC2 TXS0102DCUR, J1 USB-TYPE-C-31-M-17, J2 CON_TERMINAL_BLOCK_02-5MM, U1 XC6206P332MR, U2 RFM98W, X1 BU-SMA-H

Commit message: library update
Connections:
- net GND: no longer J1.GND_2
- net N$1: no longer J1.VBUS_2
Other:
- moved on the sheet: C1, C2, C3, C5, C6, C7, C9, U2
